File: output/pcbs/pcb.kicad_pcb (KiCad board)
At the start: 2 copper layers, 253 x 72 mm, 103 parts

Commit message: chore: ran drc
Routing:
- net GND: track 63.4 -> 83.3 mm
Changed lines of the file:
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@@
+	)
+	(segment
+		(start 67.38 49.92)
+		(end 67.38 47.38)
+		(width 0.2)
+		(layer "F.Cu")
+		(net 3)
+	)
+	(segment
+		(start 77.54 49.92)
+		(end 82.62 44.84)
+		(width 0.2)
+		(layer "F.Cu")
+		(net 3)
 	)
 	(segment
@@
 		(width 0.2)
 		(layer "F.Cu")
+		(net 3)
+	)
+	(segment
+		(start 67.38 49.92)
+		(end 77.54 49.92)
+		(width 0.2)
+		(layer "F.Cu")
